File: betaspray-pcb/servo_subsystem.kicad_sch (KiCad schematic)
At the start: 8 parts, among them J11 Conn_01x03_Pin, J12 Conn_01x03_Pin, J13 Conn_01x03_Pin, J14 Conn_01x03_Pin, J15 Conn_01x03_Pin, J16 Conn_01x03_Pin, J17 Conn_01x03_Pin, J18 Conn_01x03_Pin

Commit message: Connected Servo labels, added debug led
Parts:
- J11, J12, J13, J14, J15, J16, J17, J18: symbol betaspray_Connector:Conn_01x03_Pin -> betaspray_MCU_Espressif:Conn_01x03_Pin
Changed lines of the file:
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@@
 	)
 	(symbol
-		(lib_id "betaspray_Connector:Conn_01x03_Pin")
+		(lib_id "betaspray_MCU_Espressif:Conn_01x03_Pin")
 		(at 60.96 60.96 0)
 		(unit 1)
@@
 	)
 	(symbol
-		(lib_id "betaspray_Connector:Conn_01x03_Pin")
+		(lib_id "betaspray_MCU_Espressif:Conn_01x03_Pin")
 		(at 60.96 44.45 0)
 		(unit 1)
@@
 	)
 	(symbol
-		(lib_id "betaspray_Connector:Conn_01x03_Pin")
+		(lib_id "betaspray_MCU_Espressif:Conn_01x03_Pin")
 		(at 88.9 93.98 0)
 		(unit 1)
@@
 	)
 	(symbol
-		(lib_id "betaspray_Connector:+3.3V")
+		(lib_id "betaspray_MCU_Espressif:+3.3V")
 		(at 102.87 104.14 180)
 		(unit 1)
@@
 	)
 	(symbol
-		(lib_id "betaspray_Connector:GND")
+		(lib_id "betaspray_MCU_Espressif:GND")
 		(at 81.28 104.14 0)
 		(unit 1)
@@
 	)
 	(symbol
-		(lib_id "betaspray_Connector:Conn_01x03_Pin")
+		(lib_id "betaspray_MCU_Espressif:Conn_01x03_Pin")
 		(at 88.9 60.96 0)
 		(unit 1)
@@
 	)
 	(symbol
-		(lib_id "betaspray_Connector:Conn_01x03_Pin")
+		(lib_id "betaspray_MCU_Espressif:Conn_01x03_Pin")
 		(at 60.96 93.98 0)
 		(unit 1)
@@
 	)
 	(symbol
-		(lib_id "betaspray_Connector:Conn_01x03_Pin")
+		(lib_id "betaspray_MCU_Espressif:Conn_01x03_Pin")
 		(at 60.96 78.74 0)
 		(unit 1)
@@
 	)
 	(symbol
-		(lib_id "betaspray_Connector:Conn_01x03_Pin")
+		(lib_id "betaspray_MCU_Espressif:Conn_01x03_Pin")
 		(at 88.9 78.74 0)
 		(unit 1)
@@
 	)
 	(symbol
-		(lib_id "betaspray_Connector:Conn_01x03_Pin")
+		(lib_id "betaspray_MCU_Espressif:Conn_01x03_Pin")
 		(at 88.9 44.45 0)
 		(unit 1)
@@
 	)
 	(symbol
-		(lib_id "betaspray_Connector:GND")
+		(lib_id "betaspray_MCU_Espressif:GND")
 		(at 109.22 104.14 0)
 		(unit 1)
@@
 	)
 	(symbol
-		(lib_id "betaspray_Connector:+3.3V")
+		(lib_id "betaspray_MCU_Espressif:+3.3V")
 		(at 74.93 104.14 180)
 		(unit 1)
