File: betaspray-pcb/power_subsystem.kicad_sch (KiCad schematic)
At the start: 8 parts, among them J1 USB_C_Receptacle_USB2.0_16P, U2 LM3940IT-3.3

Commit message: Add more decoupling caps?
Parts:
- added C8: 0.1 uF, Capacitor_SMD:C_0805_2012Metric_Pad1.18x1.45mm_HandSolder, symbol betaspray_MCU_Espressif:C
- added C9: 100 uF, Capacitor_SMD:C_0805_2012Metric_Pad1.18x1.45mm_HandSolder, symbol betaspray_MCU_Espressif:C
Connections:
- net GND: now also C8.2, C9.2
- net VDD3V: now also C8.1, C9.1
Other:
- note added: "3.3V Power Status LED(?)"
- note removed: "am i stupid"
- moved on the sheet: D1, R3

Commit message: Ver0, pls'
Parts:
- renumbered J1 to e1
Changed lines of the file:
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@@
 		(dnp no)
 		(fields_autoplaced yes)
-		(property "Reference" "J1"
+		(property "Reference" "e1"
 			(at 44.45 19.05 0)
 			(effects
@@
 			(project ""
 				(path "/5d34c70f-469d-43be-b671-484e3b695429/48241481-8c99-4c08-b4b7-9ff4b52e25cf"
-					(reference "J1")
+					(reference "e1")
 					(unit 1)
 				)
