File: betaspray-pcb/betaspray-pcb.kicad_pcb (KiCad board)
At the start: 4 copper layers, 99.3 x 99.3 mm, 44 parts, among them J10 Conn_01x09_Pin, J11 Conn_01x03_Pin, J12 Conn_01x03_Pin, J13 Conn_01x03_Pin, J14 Conn_01x03_Pin, J15 Conn_01x03_Pin, J16 Conn_01x03_Pin, J17 Conn_01x03_Pin, J18 Conn_01x03_Pin, J2 Conn_01x02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

Commit message: fixed footprint
Parts:
- J10, J8: footprint Connector_TE-Connectivity:TE_826576-9_1x09_P3.96mm_Vertical -> Connector_PinHeader_2.54mm:PinHeader_1x09_P2.54mm_Vertical
- moved J10 10.7 mm to (110.0, 121.8), turned to 180 degrees
- moved J8 9.76 mm to (104.8, 121.8), turned to 180 degrees
Routing:
- net SDA: track 61.4 -> 54.0 mm
- net VS_SYNC_ROW: track 58.6 -> 52.1 mm
- net CAM_RST: track 22.9 -> 28.7 mm
- net D5: track 33.7 -> 39.5 mm
- net D7: track 37.5 -> 42.9 mm
- net D3: track 31.2 -> 36.5 mm
- net D8: track 51.8 -> 46.8 mm
- net CAM_PWR_DEL: track 39.6 -> 43.7 mm
- net D9: track 42.4 -> 46.3 mm
- net D6: track 48.8 -> 45.1 mm
- net PIXEL_CLK: track 46.5 -> 49.8 mm
- net D4: track 45.7 -> 43.5 mm
- net VS_SYNC_FRAME: track 53.9 -> 55.3 mm
