File: betaspray-pcb/betaspray-pcb.kicad_sch (KiCad schematic)
At the start: 11 parts, among them SW1 SW_Push, SW2 SW_Push, U1 ESP32-S3-WROOM-1

Commit message: Add more decoupling caps?
Connections:
- net LSR_4: now reaches U1.15 (IO3)
- net LSR_2: now reaches U1.8 (IO15)
- net LSR_3: now reaches U1.9 (IO16)
- no-connect marks 9 -> 6
Other:
- sheet servo_subsystem ports: added LSR_2, LSR_3, LSR_4; removed none
Changed lines of the file:
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@@
 	)
 	(no_connect
-		(at 74.93 55.88)
-	)
-	(no_connect
 		(at 127 45.72)
 	)
@@
 	)
 	(no_connect
-		(at 90.17 88.9)
-	)
-	(no_connect
-		(at 90.17 86.36)
-	)
-	(no_connect
 		(at 127 63.5)
 	)
@@
 		)
 	)
+	(label "LSR_3"
+		(at 90.17 88.9 180)
+		(effects
+			(font
+				(size 1.27 1.27)
+			)
+			(justify right bottom)
+		)
+	)
 	(label "EN"
 		(at 200.66 49.53 0)
@@
 		)
 	)
+	(label "LSR_4"
+		(at 74.93 55.88 180)
+		(effects
+			(font
+				(size 1.27 1.27)
+			)
+			(justify right bottom)
+		)
+	)
 	(label "SERV1"
 		(at 189.23 125.73 180)
@@
 		)
 	)
+	(label "LSR_2"
+		(at 90.17 86.36 180)
+		(effects
+			(font
+				(size 1.27 1.27)
+			)
+			(justify right bottom)
+		)
+	)
 	(label "SERV6"
 		(at 96.52 66.04 180)
@@
 		)
 	)
+	(label "LSR_2"
+		(at 215.9 129.54 0)
+		(effects
+			(font
+				(size 1.27 1.27)
+			)
+			(justify left bottom)
+		)
+	)
 	(label "SERV3"
 		(at 189.23 130.81 180)
@@
 		)
 	)
+	(label "LSR_4"
+		(at 215.9 137.16 0)
+		(effects
+			(font
+				(size 1.27 1.27)
+			)
+			(justify left bottom)
+		)
+	)
+	(label "LSR_3"
+		(at 215.9 133.35 0)
+		(effects
+			(font
+				(size 1.27 1.27)
+			)
+			(justify left bottom)
+		)
+	)
 	(label "BOOT"
 		(at 246.38 48.26 0)
@@
 			(effects
 				(font
+					(size 1.27 1.27)
+				)
+				(justify right)
+			)
+		)
+		(pin "LSR_2" input
+			(at 215.9 129.54 0)
+			(effects
+				(font
+					(size 1.27 1.27)
+				)
+				(justify right)
+			)
+		)
+		(pin "LSR_3" input
+			(at 215.9 133.35 0)
+			(effects
+				(font
+					(size 1.27 1.27)
+				)
+				(justify right)
+			)
+		)
+		(pin "LSR_4" input
+			(at 215.9 137.16 0)
+			(effects
+				(font

Commit message: Ver0, pls'
Parts:
- added H1, H2, H3, H4: MountingHole, MountingHole:MountingHole_3.2mm_M3, symbol Mechanical:MountingHole
Connections:
- net LSR_2: no longer U1.8 (IO15)
- net LSR_3: no longer U1.9 (IO16)
- net LSR_4: no longer U1.15 (IO3)
- no-connect marks 6 -> 9

Commit message: Create initial 2layer pcb, need to check
Parts:
- SBOOT: renamed from SW2; footprint Button_Switch_SMD:SW_DIP_SPSTx02_Slide_9.78x7.26mm_W8.61mm_P2.54mm -> Button_Switch_THT:SW_TH_Tactile_Omron_B3F-10xx
- SRST: renamed from SW1; footprint Button_Switch_SMD:SW_DIP_SPSTx02_Slide_9.78x7.26mm_W8.61mm_P2.54mm -> Button_Switch_THT:SW_TH_Tactile_Omron_B3F-10xx
Changed lines of the file:
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@@
 		(dnp no)
 		(fields_autoplaced yes)
-		(property "Reference" "SW2"
+		(property "Reference" "SBOOT"
 			(at 246.38 53.3399 90)
 			(effects
@@
 			)
 		)
-		(property "Footprint" "Button_Switch_SMD:SW_DIP_SPSTx02_Slide_9.78x7.26mm_W8.61mm_P2.54mm"
+		(property "Footprint" "Button_Switch_THT:SW_TH_Tactile_Omron_B3F-10xx"
 			(at 247.65 54.61 0)
 			(effects
@@
 			(project "betaspray-pcb"
 				(path "/5d34c70f-469d-43be-b671-484e3b695429"
-					(reference "SW2")
+					(reference "SBOOT")
 					(unit 1)
 				)
@@
 		(dnp no)
 		(fields_autoplaced yes)
-		(property "Reference" "SW1"
+		(property "Reference" "SRST"
 			(at 200.66 54.6099 90)
 			(effects
@@
 			)
 		)
-		(property "Footprint" "Button_Switch_SMD:SW_DIP_SPSTx02_Slide_9.78x7.26mm_W8.61mm_P2.54mm"
+		(property "Footprint" "Button_Switch_THT:SW_TH_Tactile_Omron_B3F-10xx"
 			(at 201.93 55.88 0)
 			(effects
@@
 			(project ""
 				(path "/5d34c70f-469d-43be-b671-484e3b695429"
-					(reference "SW1")
-					(unit 1)
-				)
+					(reference "SRST")
+					(unit 1)
+				)

Commit message: Fixed footprint
Parts:
- renumbered SBOOT to SBOOT1, SRST to SRST1
Changed lines of the file:
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@@
 		(dnp no)
 		(fields_autoplaced yes)
-		(property "Reference" "SBOOT"
+		(property "Reference" "SBOOT1"
 			(at 246.38 53.3399 90)
 			(effects
@@
 			(project "betaspray-pcb"
 				(path "/5d34c70f-469d-43be-b671-484e3b695429"
-					(reference "SBOOT")
+					(reference "SBOOT1")
 					(unit 1)
 				)
@@
 		(dnp no)
 		(fields_autoplaced yes)
-		(property "Reference" "SRST"
+		(property "Reference" "SRST1"
 			(at 200.66 54.6099 90)
 			(effects
@@
 			(project ""
 				(path "/5d34c70f-469d-43be-b671-484e3b695429"
-					(reference "SRST")
-					(unit 1)
-				)
+					(reference "SRST1")
+					(unit 1)
+				)
